Commit message: camera done

File: thesis_gazebo/thesis_vehicles/bluerov_heavy_defcamera_vehicle/urdf/sensors.xacro (robot description, xacro)
@@ -40,5 +40,5 @@
   <!-- Mount a camera  -->
   <xacro:default_camera namespace="${namespace}" parent_link="${namespace}/base_link" suffix="">
-    <origin xyz="0.25 0 0" rpy="0 1.57 0"/>
+    <origin xyz="0.25 0 0" rpy="0 0 0"/>
   </xacro:default_camera>
 </robot>

Commit message: pitch e roll well tuned

File: thesis_gazebo/thesis_vehicles/bluerov_heavy_defcamera_vehicle/urdf/sensors.xacro (robot description, xacro)
@@ -40,5 +40,5 @@
   <!-- Mount a camera  -->
   <xacro:default_camera namespace="${namespace}" parent_link="${namespace}/base_link" suffix="">
-    <origin xyz="0.25 0 0" rpy="0 0 0"/>
+    <origin xyz="0.25 0 0" rpy="0 0 0" mass="0"/>
   </xacro:default_camera>
 </robot>

Commit message: Update(sonar_based_localisation): First Inspection Done

File: thesis_gazebo/thesis_vehicles/bluerov_heavy_defcamera_vehicle/urdf/sensors.xacro (robot description, xacro)
@@ -54,5 +54,5 @@
               reflectivityDatabaseFile="multibeam_sonar/nps_uw_multibeam_sonar/worlds/variationalReflectivityDatabase.csv"
               robot_link="${namespace}/base_link" ray_visual="true" gaussian_noise_mean="0.0" gaussian_noise_stddev="0.02">
-    <origin xyz="0.25 0 -0.25" rpy="0 0.174532925 0"/>
+    <origin xyz="0.25 0 -0.25" rpy="0 0 0"/>
   </xacro:multibeam_blueview_p900_macro>
 </robot>
