Commit message: SONAR DONE

File: multibeam_sonar/nps_uw_multibeam_sonar/urdf/multibeam_sonar_blueview_p900.xacro (robot description, xacro)
@@ -5,5 +5,5 @@
     <link name="${name}_link">
       <inertial>
-        <mass value="4.35"/>
+        <mass value="0.0"/>
         <pose xyz="0 0 0" rpy="0 0 0"/>
         <inertia ixx="0.0360" ixy="0" ixz="0" iyy="0" iyz="0" izz="0.0360"/>

File: thesis_gazebo/thesis_vehicles/bluerov_heavy_defcamera_vehicle/urdf/sensors.xacro (robot description, xacro)
@@ -48,5 +48,5 @@
                artificialVehicleVibration constantReflectivity reflectivityDatabaseFile
                robot_link ray_visual *origin"> -->
-  <xacro:multibeam_blueview_p900_macro name="${namespace}" scale="1 1 1" gpu_ray="true" robot_name="bluerov_heavy"
+  <xacro:multibeam_blueview_p900_macro name="${namespace}" scale="0.5 0.5 0.5" gpu_ray="false" robot_name="bluerov_heavy"
               sonar_image_topic="sonar_image_topic" sonar_image_raw_topic="sonar_image_raw_topic" debug="true"
               maxDistance="20" raySkips="10" plotScaler="1" sensorGain="0.02" writeLog="false" writeFrameInterval="5"
@@ -54,5 +54,5 @@
               reflectivityDatabaseFile="multibeam_sonar/nps_uw_multibeam_sonar/worlds/variationalReflectivityDatabase.csv"
               robot_link="${namespace}/base_link" ray_visual="true" gaussian_noise_mean="0.0" gaussian_noise_stddev="0.02">
-    <origin xyz="0 0 -0.25" rpy="0 0 0"/>
+    <origin xyz="0.25 0 -0.25" rpy="0 0 0"/>
   </xacro:multibeam_blueview_p900_macro>
 </robot>

Commit message: Update: Sonar Parameters chosen

File: multibeam_sonar/nps_uw_multibeam_sonar/urdf/multibeam_sonar_blueview_p900.xacro (robot description, xacro)
@@ -35,5 +35,11 @@
         <camera>
           <!-- 90 degrees for the M900-90 -->
-          <horizontal_fov>1.57079632679</horizontal_fov>
+          <!-- <horizontal_fov>1.57079632679</horizontal_fov> -->
+          <!--30 graus-->
+          <!-- <horizontal_fov>0.523598775</horizontal_fov> -->
+          <!--45 graus-->
+          <!-- <horizontal_fov>0.785398163</horizontal_fov> -->
+          <!--60 graus-->
+          <horizontal_fov>1.047197551</horizontal_fov>
           <image>
             <width>512</width>
@@ -57,5 +63,5 @@
           <!-- Sonar properties -->
           <verticalFOV>20</verticalFOV>
-          <sonarFreq>900e3</sonarFreq>
+          <sonarFreq>1.8e6</sonarFreq>
           <bandwidth>29.9e3</bandwidth>
           <soundSpeed>1500</soundSpeed>

File: thesis_gazebo/thesis_vehicles/bluerov_heavy_defcamera_vehicle/urdf/sensors.xacro (robot description, xacro)
@@ -48,11 +48,11 @@
                artificialVehicleVibration constantReflectivity reflectivityDatabaseFile
                robot_link ray_visual *origin"> -->
-  <xacro:multibeam_blueview_p900_macro name="${namespace}" scale="0.5 0.5 0.5" gpu_ray="false" robot_name="bluerov_heavy"
+  <xacro:multibeam_blueview_p900_macro name="multibeam" scale="0.5 0.5 0.5" gpu_ray="false" robot_name="bluerov_heavy"
               sonar_image_topic="sonar_image_topic" sonar_image_raw_topic="sonar_image_raw_topic" debug="true"
-              maxDistance="20" raySkips="10" plotScaler="1" sensorGain="0.02" writeLog="false" writeFrameInterval="5"
-              artificialVehicleVibration="false" constantReflectivity="false" fidelity="500"
+              maxDistance="15" raySkips="10" plotScaler="1" sensorGain="0.02" writeLog="true" writeFrameInterval="5"
+              artificialVehicleVibration="false" constantReflectivity="true" fidelity="500"
               reflectivityDatabaseFile="multibeam_sonar/nps_uw_multibeam_sonar/worlds/variationalReflectivityDatabase.csv"
               robot_link="${namespace}/base_link" ray_visual="true" gaussian_noise_mean="0.0" gaussian_noise_stddev="0.02">
-    <origin xyz="0.25 0 -0.25" rpy="0 0 0"/>
+    <origin xyz="0.25 0 -0.25" rpy="0 0.174532925 0"/>
   </xacro:multibeam_blueview_p900_macro>
 </robot>

Commit message: Update: smooth path; working on surge controller and currents

File: multibeam_sonar/nps_uw_multibeam_sonar/urdf/multibeam_sonar_blueview_p900.xacro (robot description, xacro)
@@ -34,4 +34,6 @@
         <update_rate>10</update_rate>
         <camera>
+          <!-- 120 degrees for the M900-90 -->
+          <!-- <horizontal_fov>2.0943295102</horizontal_fov> -->
           <!-- 90 degrees for the M900-90 -->
           <!-- <horizontal_fov>1.57079632679</horizontal_fov> -->
@@ -46,5 +48,6 @@
             <!-- Set vertical FOV by setting image height -->
             <!-- Approx 2 times the spec sheet (sepc: 20 deg.) -->
-            <height>228</height>
+            <!-- <height>228</height> -->
+            <height>171</height>
             <format>R8G8B8</format>
           </image>
@@ -62,5 +65,5 @@
         <plugin filename="libnps_multibeam_sonar_ros_plugin.so" name="${name}_sensor_controller">
           <!-- Sonar properties -->
-          <verticalFOV>20</verticalFOV>
+          <verticalFOV>15</verticalFOV>
           <sonarFreq>1.8e6</sonarFreq>
           <bandwidth>29.9e3</bandwidth>

File: thesis_gazebo/thesis_vehicles/bluerov_heavy_defcamera_vehicle/urdf/sensors.xacro (robot description, xacro)
@@ -50,9 +50,9 @@
   <xacro:multibeam_blueview_p900_macro name="multibeam" scale="0.5 0.5 0.5" gpu_ray="false" robot_name="bluerov_heavy"
               sonar_image_topic="sonar_image_topic" sonar_image_raw_topic="sonar_image_raw_topic" debug="true"
-              maxDistance="15" raySkips="10" plotScaler="1" sensorGain="0.02" writeLog="true" writeFrameInterval="5"
+              maxDistance="15" raySkips="20" plotScaler="1" sensorGain="0.02" writeLog="true" writeFrameInterval="5"
               artificialVehicleVibration="false" constantReflectivity="true" fidelity="500"
               reflectivityDatabaseFile="multibeam_sonar/nps_uw_multibeam_sonar/worlds/variationalReflectivityDatabase.csv"
               robot_link="${namespace}/base_link" ray_visual="true" gaussian_noise_mean="0.0" gaussian_noise_stddev="0.02">
-    <origin xyz="0.25 0 -0.25" rpy="0 0 0"/>
+    <origin xyz="0.22 0 -0.19" rpy="0 0 0"/>
   </xacro:multibeam_blueview_p900_macro>
 </robot>

File: thesis_gazebo/thesis_vehicles/bluerov_heavy_defcamera_vehicle/urdf/snippets.xacro (robot description, xacro)
@@ -59,5 +59,5 @@
         <dynamics>
           <type>FirstOrder</type>
-          <timeConstant>0.2</timeConstant>
+          <timeConstant>0.000001</timeConstant>
         </dynamics>
         <conversion>
